Commit message: added the mujoco window viewer and saved the map of the workspace.

File: src/amr_bot/urdf/supermarketbot.urdf (robot description, URDF)
Before this commit: robot supermarketbot, 6 links, 5 joints
Links:
- link chassis_link: geometry collision box size=0.16065 0.18 0.1; collision cylinder length=0.02 radius=0.009
- link left_wheel_link: geometry collision cylinder length=0.02 radius=0.035; visual mesh filename=package://amr_bot/models/meshes/wheel.stl scale=0.001 0.001 0.001
- link lidar_link: geometry collision box size=0.06 0.06 0.06; visual cylinder length=0.015 radius=0.02
- link right_wheel_link: geometry collision cylinder length=0.02 radius=0.035; visual mesh filename=package://amr_bot/models/meshes/wheel.stl scale=0.001 0.001 0.001
